Commit message: Add rgbd_simul (publishes point cloud from bag) Modify robotino_description and robotino_simul.launch to launch rgbd_simul Modify rviz config to display point cloud Add vision package for color segmentation and sift detection and matching

File: catkin_ws/src/hardware/robot_description/robotino.urdf (robot description, URDF)
Before this commit: robot robotino, 6 links, 5 joints
Links:
- added link camera_depth_optical_frame
Joints:
- added joint depth_camera_joint: type fixed, parent base_link, child camera_depth_optical_frame, origin xyz=0 0 0.25 rpy=-1.5708 0 -1.5708

Commit message: Change topic name for the point cloud. Modify robotino.urdf robotino_simul.launch, getting_started.rviz and rgbd_simul for this change. Modify sift recognition node.

File: catkin_ws/src/hardware/robot_description/robotino.urdf (robot description, URDF)
Before this commit: robot robotino, 7 links, 6 joints
Links:
- removed link camera_depth_optical_frame
- added link camera_color_optical_frame
Joints:
- joint depth_camera_joint: child camera_depth_optical_frame -> camera_color_optical_frame; origin xyz=0 0 0.25 rpy=-1.5708 0 -1.5708 -> xyz=0 0 0.25 rpy=-1.8708 0 -1.5708

Commit message: Correct some problems with external bags

File: catkin_ws/src/hardware/robot_description/robotino.urdf (robot description, URDF)
Before this commit: robot robotino, 7 links, 6 joints
Links:
- added link camera_depth_optical_frame
Joints:
- added joint depth_camera_joint2: type fixed, parent base_link, child camera_depth_optical_frame, origin xyz=0 0 0.25 rpy=-1.8708 0 -1.5708
